File: fib_backplate.kicad_sch (KiCad schematic)
At the start: 32 parts

Commit message: moved eink connector slightly to the side, ready for fabrication v1.1
Connections:
- net RST_0: now also SV23.11, SV23.12; no longer SV23.15, SV23.16
- new net: SV23.15, SV23.16
